Commit message: Add files via upload

File: trixy.xacro (robot description, xacro)
@@ -1,3 +1,3 @@
-<?xml version="1.0"?>
+<?xml version='1.0'?>
 <robot name="trixy" xmlns:xacro="http://www.ros.org/wiki/xacro">
 <link name="casco">
@@ -5,5 +5,5 @@
 <origin xyz="0 0 0" rpy="0 -0 0" />
 <geometry>
-<mesh filename="package://trixy/urdf/casco.stl"/>
+<mesh filename="package://mergulhao/urdf/casco.stl"/>
 </geometry>
 <material name="casco_material">
@@ -14,5 +14,5 @@
 <origin xyz="0 0 0" rpy="0 -0 0" />
 <geometry>
-<mesh filename="package://trixy/urdf/casco.stl"/>
+<mesh filename="package://mergulhao/urdf/casco.stl"/>
 </geometry>
 <material name="casco_material">
@@ -30,5 +30,5 @@
 <origin xyz="7.38165e-18 0.00424822 -0.049" rpy="4.93038e-32 7.31806e-32 -6.78879e-80" />
 <geometry>
-<mesh filename="package://trixy/urdf/thruster_base.stl"/>
+<mesh filename="package://mergulhao/urdf/thruster_base.stl"/>
 </geometry>
 <material name="thruster_base_material">
@@ -39,5 +39,5 @@
 <origin xyz="7.38165e-18 0.00424822 -0.049" rpy="4.93038e-32 7.31806e-32 -6.78879e-80" />
 <geometry>
-<mesh filename="package://trixy/urdf/thruster_base.stl"/>
+<mesh filename="package://mergulhao/urdf/thruster_base.stl"/>
 </geometry>
 <material name="thruster_base_material">
@@ -51,9 +51,17 @@
 </inertial>
 </link>
+<joint name="casco_thruster" type="fixed">
+<origin xyz="-0.00420826 -2.44379e-10 -0.12" rpy="7.66335e-47 1.31372e-46 -1.5708" />
+<parent link="casco" />
+<child link="thruster_base" />
+<axis xyz="0 0 1"/>
+<limit effort="1" velocity="20" />
+<joint_properties friction="0.0"/>
+</joint>
 <link name="thruster_helice">
 <visual>
 <origin xyz="-7.08857e-17 -5.55112e-16 -0.009842" rpy="-1.5708 5.84663e-16 -1.75162e-46" />
 <geometry>
-<mesh filename="package://trixy/urdf/thruster_helice.stl"/>
+<mesh filename="package://mergulhao/urdf/thruster_helice.stl"/>
 </geometry>
 <material name="thruster_helice_material">
@@ -64,5 +72,5 @@
 <origin xyz="-7.08857e-17 -5.55112e-16 -0.009842" rpy="-1.5708 5.84663e-16 -1.75162e-46" />
 <geometry>
-<mesh filename="package://trixy/urdf/thruster_helice.stl"/>
+<mesh filename="package://mergulhao/urdf/thruster_helice.stl"/>
 </geometry>
 <material name="thruster_helice_material">
@@ -84,17 +92,9 @@
 <joint_properties damping ="0.0" friction="0.0"/>
 </joint>
-<joint name="casco_thruster" type="fixed">
-<origin xyz="-0.00420826 -2.44379e-10 -0.12" rpy="7.66335e-47 1.31372e-46 -1.5708" />
-<parent link="casco" />
-<child link="thruster_base" />
-<axis xyz="0 0 1"/>
-<limit effort="1" velocity="20" />
-<joint_properties friction="0.0"/>
-</joint>
 <link name="sonar_ping360">
 <visual>
 <origin xyz="0 0.00135122 -0.0401341" rpy="-1.5708 -0 0" />
 <geometry>
-<mesh filename="package://trixy/urdf/sonar_ping360.stl"/>
+<mesh filename="package://mergulhao/urdf/sonar_ping360.stl"/>
 </geometry>
 <material name="sonar_ping360_material">
@@ -105,5 +105,5 @@
 <origin xyz="0 0.00135122 -0.0401341" rpy="-1.5708 -0 0" />
 <geometry>
-<mesh filename="package://trixy/urdf/sonar_ping360.stl"/>
+<mesh filename="package://mergulhao/urdf/sonar_ping360.stl"/>
 </geometry>
 <material name="sonar_ping360_material">
@@ -129,5 +129,5 @@
 <origin xyz="0 0 0" rpy="3.14159 -0 0" />
 <geometry>
-<mesh filename="package://trixy/urdf/penetrator_sonar.stl"/>
+<mesh filename="package://mergulhao/urdf/penetrator_sonar.stl"/>
 </geometry>
 <material name="penetrator_sonar_material">
@@ -138,5 +138,5 @@
 <origin xyz="0 0 0" rpy="3.14159 -0 0" />
 <geometry>
-<mesh filename="package://trixy/urdf/penetrator_sonar.stl"/>
+<mesh filename="package://mergulhao/urdf/penetrator_sonar.stl"/>
 </geometry>
 <material name="penetrator_sonar_material">
@@ -162,5 +162,5 @@
 <origin xyz="8.753e-05 -0.000210673 -0.016" rpy="0 -0 0" />
 <geometry>
-<mesh filename="package://trixy/urdf/nut_thruster.stl"/>
+<mesh filename="package://mergulhao/urdf/nut_thruster.stl"/>
 </geometry>
 <material name="nut_thruster_material">
@@ -171,5 +171,5 @@
 <origin xyz="8.753e-05 -0.000210673 -0.016" rpy="0 -0 0" />
 <geometry>
-<mesh filename="package://trixy/urdf/nut_thruster.stl"/>
+<mesh filename="package://mergulhao/urdf/nut_thruster.stl"/>
 </geometry>
 <material name="nut_thruster_material">
@@ -195,5 +195,5 @@
 <origin xyz="0 0 0" rpy="3.14159 -0 0" />
 <geometry>
-<mesh filename="package://trixy/urdf/penetrator_thruster.stl"/>
+<mesh filename="package://mergulhao/urdf/penetrator_thruster.stl"/>
 </geometry>
 <material name="penetrator_thruster_material">
@@ -204,5 +204,5 @@
 <origin xyz="0 0 0" rpy="3.14159 -0 0" />
 <geometry>
-<mesh filename="package://trixy/urdf/penetrator_thruster.stl"/>
+<mesh filename="package://mergulhao/urdf/penetrator_thruster.stl"/>
 </geometry>
 <material name="penetrator_thruster_material">
@@ -228,5 +228,5 @@
 <origin xyz="-0.000226036 -2.95444e-05 0" rpy="3.14159 -0 0" />
 <geometry>
-<mesh filename="package://trixy/urdf/nut_sonar.stl"/>
+<mesh filename="package://mergulhao/urdf/nut_sonar.stl"/>
 </geometry>
 <material name="nut_sonar_material">
@@ -237,5 +237,5 @@
 <origin xyz="-0.000226036 -2.95444e-05 0" rpy="3.14159 -0 0" />
 <geometry>
-<mesh filename="package://trixy/urdf/nut_sonar.stl"/>
+<mesh filename="package://mergulhao/urdf/nut_sonar.stl"/>
 </geometry>
 <material name="nut_sonar_material">
@@ -261,5 +261,5 @@
 <origin xyz="0 0 0.0525" rpy="-1.5708 -0 0" />
 <geometry>
-<mesh filename="package://trixy/urdf/eixo_flap_base.stl"/>
+<mesh filename="package://mergulhao/urdf/eixo_flap_base.stl"/>
 </geometry>
 <material name="eixo_flap_base_material">
@@ -270,5 +270,5 @@
 <origin xyz="0 0 0.0525" rpy="-1.5708 -0 0" />
 <geometry>
-<mesh filename="package://trixy/urdf/eixo_flap_base.stl"/>
+<mesh filename="package://mergulhao/urdf/eixo_flap_base.stl"/>
 </geometry>
 <material name="eixo_flap_base_material">
@@ -290,174 +290,9 @@
 <joint_properties friction="0.0"/>
 </joint>
-<link name="eixo_flap">
-<visual>
-<origin xyz="0 0 -0.0245" rpy="1.5708 -0 0" />
-<geometry>
-<mesh filename="package://trixy/urdf/eixo_flap.stl"/>
-</geometry>
-<material name="eixo_flap_material">
-<color rgba="0.647059 0.647059 0.647059 1.0"/>
-</material>
-</visual>
-<collision>
-<origin xyz="0 0 -0.0245" rpy="1.5708 -0 0" />
-<geometry>
-<mesh filename="package://trixy/urdf/eixo_flap.stl"/>
-</geometry>
-<material name="eixo_flap_material">
-<color rgba="0.647059 0.647059 0.647059 1.0"/>
-</material>
-</collision>
-<inertial>
-<origin xyz="-4.61583e-10 2.86529e-06 -0.0237059" rpy="0 0 0"/>
-<mass value="0.0104144" />
-<inertia ixx="2.92663e-05" ixy="3.198e-14"  ixz="2.12095e-13" iyy="2.92663e-05" iyz="-2.63433e-09" izz="1.16968e-08" />
-</inertial>
-</link>
-<link name="flap">
-<visual>
-<origin xyz="0 0 -0.1005" rpy="-1.5708 -0 0" />
-<geometry>
-<mesh filename="package://trixy/urdf/flap.stl"/>
-</geometry>
-<material name="flap_material">
-<color rgba="0.615686 0.811765 0.929412 1.0"/>
-</material>
-</visual>
-<collision>
-<origin xyz="0 0 -0.1005" rpy="-1.5708 -0 0" />
-<geometry>
-<mesh filename="package://trixy/urdf/flap.stl"/>
-</geometry>
-<material name="flap_material">
-<color rgba="0.615686 0.811765 0.929412 1.0"/>
-</material>
-</collision>
-<inertial>
-<origin xyz="-0.0185575 1.76413e-07 -0.0655618" rpy="0 0 0"/>
-<mass value="0.0620715" />
-<inertia ixx="7.85311e-05" ixy="1.41447e-10"  ixz="4.11493e-06" iyy="9.76631e-05" iyz="-6.03888e-11" izz="2.12594e-05" />
-</inertial>
-</link>
-<link name="pç_flap">
-<visual>
-<origin xyz="0.0212557 -0.000679749 -0.003" rpy="0 -8.75812e-47 0" />
-<geometry>
-<mesh filename="package://trixy/urdf/pç_flap.stl"/>
-</geometry>
-<material name="pç_flap_material">
-<color rgba="0.615686 0.811765 0.929412 1.0"/>
-</material>
-</visual>
-<collision>
-<origin xyz="0.0212557 -0.000679749 -0.003" rpy="0 -8.75812e-47 0" />
-<geometry>
-<mesh filename="package://trixy/urdf/pç_flap.stl"/>
-</geometry>
-<material name="pç_flap_material">
-<color rgba="0.615686 0.811765 0.929412 1.0"/>
-</material>
-</collision>
-<inertial>
-<origin xyz="0.0167347 -0.000679749 -0.0015" rpy="0 0 0"/>
-<mass value="0.000621423" />
-<inertia ixx="4.85566e-09" ixy="0"  ixz="2.35806e-54" iyy="2.78564e-08" iyz="0" izz="3.17799e-08" />
-</inertial>
-</link>
-<joint name="pç_flap_l" type="fixed">
-<origin xyz="-0.0212557 0.000679749 0.0045" rpy="0 -4.93038e-31 0" />
-<parent link="flap" />
-<child link="pç_flap" />
-<axis xyz="0 0 1"/>
-<limit effort="1" velocity="20" />
-<joint_properties friction="0.0"/>
-</joint>
-<joint name="ex_flp_l" type="fixed">
-<origin xyz="0 0 -0.1155" rpy="3.14159 -0 3.14159" />
-<parent link="eixo_flap" />
-<child link="flap" />
-<axis xyz="0 0 1"/>
-<limit effort="1" velocity="20" />
-<joint_properties friction="0.0"/>
-</joint>
-<link name="gaxeta">
-<visual>
-<origin xyz="0 0 0" rpy="3.14159 -0 0" />
-<geometry>
-<mesh filename="package://trixy/urdf/gaxeta.stl"/>
-</geometry>
-<material name="gaxeta_material">
-<color rgba="0.615686 0.811765 0.929412 1.0"/>
-</material>
-</visual>
-<collision>
-<origin xyz="0 0 0" rpy="3.14159 -0 0" />
-<geometry>
-<mesh filename="package://trixy/urdf/gaxeta.stl"/>
-</geometry>
-<material name="gaxeta_material">
-<color rgba="0.615686 0.811765 0.929412 1.0"/>
-</material>
-</collision>
-<inertial>
-<origin xyz="-2.39888e-11 -4.38898e-05 -0.00300727" rpy="0 0 0"/>
-<mass value="0.00144054" />
-<inertia ixx="9.39445e-09" ixy="1.49997e-15"  ixz="-3.17149e-16" iyy="1.0572e-08" iyz="6.64662e-11" izz="1.03195e-08" />
-</inertial>
-</link>
-<link name="borracha_eixo">
-<visual>
-<origin xyz="0 0 0" rpy="1.5708 -0 0" />
-<geometry>
-<mesh filename="package://trixy/urdf/borracha_eixo.stl"/>
-</geometry>
-<material name="borracha_eixo_material">
-<color rgba="0.917647 0.917647 0.917647 1.0"/>
-</material>
-</visual>
-<collision>
-<origin xyz="0 0 0" rpy="1.5708 -0 0" />
-<geometry>
-<mesh filename="package://trixy/urdf/borracha_eixo.stl"/>
-</geometry>
-<material name="borracha_eixo_material">
-<color rgba="0.917647 0.917647 0.917647 1.0"/>
-</material>
-</collision>
-<inertial>
-<origin xyz="1.2211e-19 -3.65887e-19 -0.001" rpy="0 0 0"/>
-<mass value="8.94176e-05" />
-<inertia ixx="4.55937e-10" ixy="0"  ixz="0" iyy="4.55937e-10" iyz="0" izz="8.52261e-10" />
-</inertial>
-</link>
-<joint name="bch_l" type="fixed">
-<origin xyz="0 0 0" rpy="3.14159 -0 0" />
-<parent link="gaxeta" />
-<child link="borracha_eixo" />
-<axis xyz="0 0 1"/>
-<limit effort="1" velocity="20" />
-<joint_properties friction="0.0"/>
-</joint>
-<joint name="gaxeta_l" type="fixed">
-<origin xyz="0 0 0.0506" rpy="3.14159 -0 0" />
-<parent link="eixo_flap" />
-<child link="gaxeta" />
-<axis xyz="0 0 1"/>
-<limit effort="1" velocity="20" />
-<joint_properties friction="0.0"/>
-</joint>
-<joint name="flap_l" type="revolute">
-<origin xyz="-0.0627976 -0.0852 -0.0364809" rpy="-1.5708 -0 0" />
-<parent link="casco" />
-<child link="eixo_flap" />
-<axis xyz="0 0 1"/>
-<limit effort="1" velocity="20" lower="0" upper="1.5708"/>
-<joint_properties friction="0.0"/>
-</joint>
 <link name="eixo_flap_base_2">
 <visual>
 <origin xyz="0 0 0.0525" rpy="-1.5708 1.51929e-63 0" />
 <geometry>
-<mesh filename="package://trixy/urdf/eixo_flap_base.stl"/>
+<mesh filename="package://mergulhao/urdf/eixo_flap_base.stl"/>
 </geometry>
 <material name="eixo_flap_base_material">
@@ -468,5 +303,5 @@
 <origin xyz="0 0 0.0525" rpy="-1.5708 1.51929e-63 0" />
 <geometry>
-<mesh filename="package://trixy/urdf/eixo_flap_base.stl"/>
+<mesh filename="package://mergulhao/urdf/eixo_flap_base.stl"/>
 </geometry>
 <material name="eixo_flap_base_material">
@@ -488,174 +323,9 @@
 <joint_properties friction="0.0"/>
 </joint>
-<link name="eixo_flap_2">
-<visual>
-<origin xyz="0 0 -0.0245" rpy="1.5708 5.94329e-47 0" />
-<geometry>
-<mesh filename="package://trixy/urdf/eixo_flap.stl"/>
-</geometry>
-<material name="eixo_flap_material">
-<color rgba="0.647059 0.647059 0.647059 1.0"/>
-</material>
-</visual>
-<collision>
-<origin xyz="0 0 -0.0245" rpy="1.5708 5.94329e-47 0" />
-<geometry>
-<mesh filename="package://trixy/urdf/eixo_flap.stl"/>
-</geometry>
-<material name="eixo_flap_material">
-<color rgba="0.647059 0.647059 0.647059 1.0"/>
-</material>
-</collision>
-<inertial>
-<origin xyz="-4.61583e-10 2.86529e-06 -0.0237059" rpy="0 0 0"/>
-<mass value="0.0104144" />
-<inertia ixx="2.92663e-05" ixy="3.198e-14"  ixz="2.12095e-13" iyy="2.92663e-05" iyz="-2.63433e-09" izz="1.16968e-08" />
-</inertial>
-</link>
-<link name="gaxeta_2">
-<visual>
-<origin xyz="0 -6.93889e-18 0" rpy="3.14159 -1.75162e-46 0" />
-<geometry>
-<mesh filename="package://trixy/urdf/gaxeta.stl"/>
-</geometry>
-<material name="gaxeta_material">
-<color rgba="0.615686 0.811765 0.929412 1.0"/>
-</material>
-</visual>
-<collision>
-<origin xyz="0 -6.93889e-18 0" rpy="3.14159 -1.75162e-46 0" />
-<geometry>
-<mesh filename="package://trixy/urdf/gaxeta.stl"/>
-</geometry>
-<material name="gaxeta_material">
-<color rgba="0.615686 0.811765 0.929412 1.0"/>
-</material>
-</collision>
-<inertial>
-<origin xyz="-2.39888e-11 -4.38898e-05 -0.00300727" rpy="0 0 0"/>
-<mass value="0.00144054" />
-<inertia ixx="9.39445e-09" ixy="1.49997e-15"  ixz="-3.17149e-16" iyy="1.0572e-08" iyz="6.64662e-11" izz="1.03195e-08" />
-</inertial>
-</link>
-<link name="borracha_eixo_2">
-<visual>
-<origin xyz="0 -6.93889e-18 -0.002" rpy="-1.5708 -1.75162e-46 0" />
-<geometry>
-<mesh filename="package://trixy/urdf/borracha_eixo.stl"/>
-</geometry>
-<material name="borracha_eixo_material">
-<color rgba="0.917647 0.917647 0.917647 1.0"/>
-</material>
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